Commit message: revised ik

File: urdf/M_lrmate_with_unijoint_hand.urdf (robot description, URDF)
Before this commit: robot LRMate_with_EndEffector, 11 links, 10 joints
Links:
- removed link gripper_hand
- removed link gripper_leftfinger
- removed link gripper_rightfinger
- added link wrist
Joints:
- removed joint finger_joint1
- removed joint finger_joint2
- joint joint_4: origin xyz=0.035   0.000   0.000 rpy=-1.5707963267948966    0.0000000000000000    0.0000000000000000 -> xyz=0.035   0.000   0.000 rpy=-1.5707963267948966    -0.52359877    0.0000000000000000
- joint joint_5: origin xyz=0.000   0.000  -0.420 rpy=1.5707963267948966    0.0000000000000000    0.0000000000000000 -> xyz=0.000   0.000  -0.420 rpy=1.5707963267948966    0.52359877    0.0000000000000000
- joint joint_7: child gripper_hand -> wrist
